Commit message: yellow arm link & joint wireframe

File: yellow_arm_description/urdf/base_model.urdf (robot description, URDF)
Before this commit: robot test_arm, 4 links, 3 joints
Links:
- added link end_effector
- added link gripper; visual box size=0.07 0.05 0.024
- added link link4; visual box size=0.055 0.1 0.024
- link base: geometry visual cylinder length=.05 radius=.05
- link link1: geometry visual cylinder length=.015 radius=.04
- link link2: geometry visual box size=0.055 0.145 0.025
- link link3: geometry visual box size=0.025 0.145 0.025
Joints:
- added joint joint4: type revolute, parent link3, child link4, origin xyz=0.00 0.145 0.0 rpy=0 0 0, axis 1.0 0.0 0.0, limit lower=-1.57 upper=1.57 effort=30 velocity=1.0
- added joint joint5: type revolute, parent link4, child gripper, origin xyz=0.0 0.1 0.0 rpy=0 0 0, axis 0 1.0 0.0, limit lower=-1.57 upper=1.57 effort=30 velocity=1.0
- added joint joint6: type fixed, parent gripper, child end_effector, origin xyz=0.0 0.05 0.0 rpy=0 0 0
- joint joint1: origin xyz=0 0 0.0 rpy=0 0 0 -> xyz=0 0 0.05 rpy=0 0 0
- joint joint2: origin xyz=0.0 0 0.1 rpy=0 0 0 -> xyz=0.0 0.0 0.025 rpy=0 0 0
- joint joint3: origin xyz=0.00 0.3 0.0 rpy=0 0 0 -> xyz=0.00 0.145 0.0 rpy=0 0 0
